Commit message: 0412

File: motor_control/install/small_arm_moveit_config/share/small_arm_moveit_config/config/small_arm.ros2_control.xacro (robot description, xacro)
@@ -1,77 +1,54 @@
 <?xml version="1.0"?>
 <robot xmlns:xacro="http://www.ros.org/wiki/xacro">
-    <xacro:macro name="small_arm_ros2_control" params="name initial_positions_file ros2_control_hardware_type">
+    <xacro:macro name="small_arm_ros2_control" params="name initial_positions_file">
         <xacro:property name="initial_positions" value="${load_yaml(initial_positions_file)['initial_positions']}"/>
         <ros2_control name="${name}" type="system">
             <hardware>
-                <xacro:if value="${ros2_control_hardware_type == 'fake'}">
-                    <plugin>mock_components/GenericSystem</plugin>
-                </xacro:if>
-                <xacro:if value="${ros2_control_hardware_type == 'real'}">
-                    <plugin>dynamixel_hardware/DynamixelHardware</plugin>
-                    <param name="usb_port">/dev/ttyUSB0</param>
-                    <param name="baud_rate">115200</param>
-                    <param name="use_dummy">true</param>
-                </xacro:if>
+                <!-- By default, set up controllers for simulation. This won't work on real hardware -->
+                <plugin>mock_components/GenericSystem</plugin>
             </hardware>
-      <joint name="joint1">
-        <param name="id">1</param>
-        <command_interface name="position"/>
-        <command_interface name="velocity"/>
-        <state_interface name="position"/>
-        <state_interface name="velocity"/>
-        <state_interface name="effort"/>
-      </joint>
-      <joint name="joint2">
-        <param name="id">2</param>
-        <command_interface name="position"/>
-        <command_interface name="velocity"/>
-        <state_interface name="position"/>
-        <state_interface name="velocity"/>
-        <state_interface name="effort"/>
-      </joint>
-      <joint name="joint3">
-        <param name="id">3</param>
-        <command_interface name="position"/>
-        <command_interface name="velocity"/>
-        <state_interface name="position"/>
-        <state_interface name="velocity"/>
-        <state_interface name="effort"/>
-      </joint>
-      <joint name="joint4">
-        <param name="id">4</param>
-        <command_interface name="position"/>
-        <command_interface name="velocity"/>
-        <state_interface name="position"/>
-        <state_interface name="velocity"/>
-        <state_interface name="effort"/>
-      </joint>
-      <joint name="joint5">
-        <param name="id">5</param>
-        <command_interface name="position"/>
-        <command_interface name="velocity"/>
-        <state_interface name="position"/>
-        <state_interface name="velocity"/>
-        <state_interface name="effort"/>
-      </joint>
-      <joint name="joint6">
-        <param name="id">6</param>
-        <command_interface name="position"/>
-        <command_interface name="velocity"/>
-        <state_interface name="position"/>
-        <state_interface name="velocity"/>
-        <state_interface name="effort"/>
-      </joint>
-      <joint name="gripper_joint1">
-        <param name="id">7</param>
-        <command_interface name="position"/>
-        <command_interface name="velocity"/>
-        <state_interface name="position"/>
-        <state_interface name="velocity"/>
-        <state_interface name="effort"/>
-      </joint>
-            <!-- <joint name="gripper_joint2">
-                <param name="mimic">gripper_joint1</param>
-                <param name="multiplier">-1</param>
+            <joint name="joint1">
+                <command_interface name="position"/>
+                <state_interface name="position">
+                  <param name="initial_value">${initial_positions['joint1']}</param>
+                </state_interface>
+                <state_interface name="velocity"/>
+            </joint>
+            <joint name="joint2">
+                <command_interface name="position"/>
+                <state_interface name="position">
+                  <param name="initial_value">${initial_positions['joint2']}</param>
+                </state_interface>
+                <state_interface name="velocity"/>
+            </joint>
+            <joint name="joint3">
+                <command_interface name="position"/>
+                <state_interface name="position">
+                  <param name="initial_value">${initial_positions['joint3']}</param>
+                </state_interface>
+                <state_interface name="velocity"/>
+            </joint>
+            <joint name="joint4">
+                <command_interface name="position"/>
+                <state_interface name="position">
+                  <param name="initial_value">${initial_positions['joint4']}</param>
+                </state_interface>
+                <state_interface name="velocity"/>
+            </joint>
+            <joint name="joint5">
+                <command_interface name="position"/>
+                <state_interface name="position">
+                  <param name="initial_value">${initial_positions['joint5']}</param>
+                </state_interface>
+                <state_interface name="velocity"/>
+            </joint>
+            <joint name="joint6">
+                <command_interface name="position"/>
+                <state_interface name="position">
+                  <param name="initial_value">${initial_positions['joint6']}</param>
+                </state_interface>
+                <state_interface name="velocity"/>
+            </joint>
+            <joint name="gripper_joint1">
                 <command_interface name="position"/>
                 <state_interface name="position">
@@ -79,5 +56,5 @@
                 </state_interface>
                 <state_interface name="velocity"/>
-            </joint> -->
+            </joint>
         </ros2_control>
     </xacro:macro>

File: motor_control/install/small_arm_moveit_config/share/small_arm_moveit_config/config/small_arm.urdf.xacro (robot description, xacro)
@@ -2,9 +2,8 @@
 <robot xmlns:xacro="http://www.ros.org/wiki/xacro" name="small_arm">
     <xacro:arg name="initial_positions_file" default="initial_positions.yaml" />
-    <xacro:arg name="ros2_control_hardware_type" default="fake" />
     <!-- Import small_arm urdf file -->
     <xacro:include filename="$(find small_arm_description)/urdf/small_arm.urdf.xacro" />
     <!-- Import control_xacro -->
     <xacro:include filename="small_arm.ros2_control.xacro" />
-    <xacro:small_arm_ros2_control name="FakeSystem" initial_positions_file="$(arg initial_positions_file)" ros2_control_hardware_type="$(arg ros2_control_hardware_type)"/>
+    <xacro:small_arm_ros2_control name="FakeSystem" initial_positions_file="$(arg initial_positions_file)"/>
 </robot>
